File: melexisToFcamera4layer/melexisToFcamera4layer.sch (KiCad schematic (older format))
At the start: 104 parts, among them J1 Conn_01x01, J10 Conn_01x04, J11 Conn_01x04, J2 Conn_01x01, J3 Conn_01x01, J4 Conn_01x02, J5 Conn_01x01, J6 Conn_01x02, J7 Conn_01x01, J8 Conn_01x01, J9 Conn_01x04, U1 LM27762, U2 ADP2164, U3 MLX75023, U4 MIC23050_SYML, U5 Cmod_A7, U6 MIC23050_GYML, U7 MIC23050_GYML, U8 MLX75123

Commit message: Improved schematics, prepared layout for routing
Parts:
- removed C16: 4u7, Capacitors_SMD:C_0603, symbol Device:C
- added CP2: 4u7, Capacitors_SMD:C_0603, symbol Device:CP
- added J12: Conn_01x22, symbol Connector_Generic:Conn_01x22
- added J13: Conn_01x02, Pin_Headers:Pin_Header_Straight_1x02_Pitch2.54mm, symbol Connector_Generic:Conn_01x02
- renumbered C1 to CP1, C10 to CP10, C19 to CP19, C21 to CP21, C25 to CP25, C5 to CP5, C6 to CP6
Connections:
- net +5V: now also J4.1 (Pin_1)
- net AVDD3V3: now also CP2.1
- net CLK_IN: now also J12.17 (Pin_17)
- net DATA0: now also J12.5 (Pin_5)
- net DATA1: now also J12.6 (Pin_6)
- net DATA10: now also J12.15 (Pin_15)
- net DATA11: now also J12.16 (Pin_16)
- net DATA2: now also J12.7 (Pin_7)
- net DATA3: now also J12.8 (Pin_8)
- net DATA4: now also J12.9 (Pin_9)
- net DATA5: now also J12.10 (Pin_10)
- net DATA6: now also J12.11 (Pin_11)
- net DATA7: now also J12.12 (Pin_12)
- net DATA8: now also J12.13 (Pin_13)
- net DATA9: now also J12.14 (Pin_14)
- net FSYNC: now also J12.3 (Pin_3)
- net GND: now also CP2.2
- net HSYNC: now also J12.2 (Pin_2)
- net PIXCLK: now also J12.4 (Pin_4)
- net QUIET: now also J12.18 (Pin_18)
- net RESET: now also J12.19 (Pin_19)
- net SCL: now also J12.21 (Pin_21)
- net SDA: now also J12.22 (Pin_22)
- net TRIGGER: now also J12.20 (Pin_20)
- net VDD1V8: now also C42.1, C43.1, J7.1 (Pin_1), L5.2, U6.4 (SNS)
- net VDD1V8_clean: now also C53.1, C55.1, J8.1 (Pin_1), L6.2, U7.4 (SNS)
- net VDD3V3: no longer C42.1, C43.1, C53.1, C55.1, J7.1 (Pin_1), J8.1 (Pin_1), L5.2, L6.2, U6.4 (SNS), U7.4 (SNS)
- net VSYNC: now also J12.1 (Pin_1)
- net at U5.24 (VU): now also J13.1 (Pin_1), J13.2 (Pin_2); no longer J4.1 (Pin_1)
Other:
- moved on the sheet: J4
